File: drawing/esp32_main/esp32_main.kicad_sch (KiCad schematic)
At the start: 4 parts, among them U1_Master ESP32-WROOM-32, U2_Slave ESP32-WROOM-32, U3 MAX3485, U4 MAX3485

Commit message: kicad update
Parts:
- added Q1: 2N2219, Package_TO_SOT_THT:TO-39-3, symbol Transistor_BJT:2N2219
- added SW1: SW_Push, symbol Switch:SW_Push
- added SW2: SW_Push_Open, symbol Switch:SW_Push_Open
- added U1: AM26LS31CN, Package_DIP:DIP-16_W7.62mm, symbol Interface:AM26LS31CN
- added U2: (no value), symbol GlasAutoma]:T6_Drive
Connections:
- net +5V: now reaches U2_Slave.2 (VDD)
- net +5V: now also U1_Master.2 (VDD)
- net at U3.5 (GND): now also U4.5 (GND)
- net at U3.6 (A): now also U4.6 (A)
- net at U3.7 (B): now also U4.7 (B)
- net at U1_Master.30 (IO18): now also Q1.2 (B)
- new net: SW2.1 (A), U2. (CN5(RS232))
- new net: Q1.3 (C), U2. (CN5(RS232))
- new net +12V: U2. (CN5(RS232))
- new net GND: Q1.1 (E), SW2.2 (B)
Other:
- moved on the sheet: U1_Master, U3, U4

Commit message: drawing udpate
Parts:
- added SW1A1: SW_NC_LIMIT_SWITCH_1, symbol Switch:SW_Push_Open
- added SW1A2: SW_NC_LIMIT_SWITCH_2, symbol Switch:SW_Push_Open
- added SW2: BTN_NO_START, symbol Switch:SW_Push
- added SW3: BTN_NO_STOP, symbol Switch:SW_Push
- added SW4: BTN_NO_RESET_ALARM, symbol Switch:SW_Push
- SW1A: renamed from SW2; value SW_Push_Open -> SW_NC_EM_STOP
- SW1B: renamed from SW1; value SW_Push -> SW_NO_EM_STOP
Connections:
- net at U2_Slave.14 (IO12): now also SW1B.1
- net GND_1: now reaches U3.5 (GND), U4.5 (GND)
- net A: now reaches U3.6 (A), U4.6 (A)
- net B: now reaches U3.7 (B), U4.7 (B)
Other:
- moved on the sheet: SW1A, SW1B

Commit message: adjusting drawing
Connections:
- net GND: now also SW1A1.2 (B)
- net at SW1A1.1 (A): now also U2. (CN5(RS232))
Changed lines of the file:
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@@
+	)
+	(junction
+		(at 153.67 163.83)
+		(diameter 0)
+		(color 0 0 0 0)
 	)
 	(junction
@@
 	(wire
 		(pts
+			(xy 91.44 154.94) (xy 99.06 154.94)
+		)
+		(stroke
+			(width 0)
+			(type default)
+		)
+	)
+	(wire
+		(pts
 			(xy 68.58 115.57) (xy 68.58 38.1)
 		)
@@
 	(wire
 		(pts
+			(xy 109.22 154.94) (xy 153.67 154.94)
+		)
+		(stroke
+			(width 0)
+			(type default)
+		)
+	)
+	(wire
+		(pts
 			(xy 124.46 83.82) (xy 217.17 83.82)
 		)
@@
 	(wire
 		(pts
-			(xy 128.27 163.83) (xy 156.21 163.83)
+			(xy 128.27 163.83) (xy 153.67 163.83)
+		)
+		(stroke
+			(width 0)
+			(type default)
+		)
+	)
+	(wire
+		(pts
+			(xy 91.44 175.26) (xy 91.44 154.94)
 		)
 		(stroke
@@
 	(wire
 		(pts
+			(xy 153.67 154.94) (xy 153.67 163.83)
+		)
+		(stroke
+			(width 0)
+			(type default)
+		)
+	)
+	(wire
+		(pts
 			(xy 124.46 115.57) (xy 124.46 83.82)
 		)
@@
 		)
 		(stroke
+			(width 0)
+			(type default)
+		)
+	)
+	(wire
+		(pts
+			(xy 153.67 163.83) (xy 156.21 163.83)
+		)
+		(stroke
